Commit message: Included the panda hand and fingers into the khi library to see if it can facilitate obstacle avoidance method.

File: scripts/assets/urdf/RS007/rs007l_panda.urdf (robot description, URDF)
Before this commit: robot rs007l, 10 links, 9 joints
Links:
- link base_link: geometry collision mesh filename=meshes/RS007L_J0.stl; visual mesh filename=meshes/RS007L_J0.stl
- link link1: geometry collision mesh filename=meshes/RS007L_J1.stl; visual mesh filename=meshes/RS007L_J1.stl
- link link2: geometry collision mesh filename=meshes/RS007L_J2.stl; visual mesh filename=meshes/RS007L_J2.stl
- link link3: geometry collision mesh filename=meshes/RS007L_J3.stl; visual mesh filename=meshes/RS007L_J3.stl
- link link4: geometry collision mesh filename=meshes/RS007L_J4.stl; visual mesh filename=meshes/RS007L_J4.stl
- link link5: geometry collision mesh filename=meshes/RS007L_J5.stl; visual mesh filename=meshes/RS007L_J5.stl
- link link6: geometry collision mesh filename=meshes/RS007L_J6.stl; visual mesh filename=meshes/RS007L_J6.stl
- link panda_hand: geometry collision mesh filename=../franka_description/meshes/collision/hand.obj; visual mesh filename=../franka_description/meshes/visual/hand.dae
- link panda_leftfinger: geometry collision mesh filename=../franka_description/meshes/collision/finger.obj; visual mesh filename=../franka_description/meshes/visual/finger.dae
- link panda_rightfinger: geometry collision mesh filename=../franka_description/meshes/collision/finger.obj; visual mesh filename=../franka_description/meshes/visual/finger.dae

Commit message: Successfully embedded moveit-based planner and controller to the project.

File: scripts/assets/urdf/RS007/rs007l_panda.urdf (robot description, URDF)
Before this commit: robot rs007l, 10 links, 9 joints
Links:
- added link weld_tip
Joints:
- added joint weld_tip_fixed: type fixed, parent panda_hand, child weld_tip, origin xyz=0 0 0.1 rpy=0 0 0
