Commit message: ROS synchronous planning done with collision avoidance constraints for each robot, resulting a feasible solution.

File: scripts/assets/urdf/big_part.urdf (robot description, URDF)
Before this commit: robot big_part_robot, 2 links, 1 joints
Links:
- link link1: geometry collision box size=0.04 0.04 0.04; visual box size=0.04 0.04 0.04
Joints:
- joint base_to_link1: origin xyz=0 0 0.015 rpy=0 0 0 -> xyz=0 0 0.025 rpy=0 0 0
